File: Ground_Station_Electronics/Ground_Station_Electronics.kicad_pcb (KiCad board)
At the start: 2 copper layers, 35 parts, among them J1 RJ45_Shielded_Labelled, J2 ARGB_Header, M1 Motor_Servo, M2 Motor_Servo, U1 LM2576HVS-5, U2 Teensy_4.1, U3 Adafruit_GPS_V3, U4 BNO055_Adafruit_Breakout, U5 RFM95W_Adafruit_Breakout, U6 MAX3488E, U7 SN74AHCT125D

Commit message: design rules and grouping
Parts:
- removed C6, C7: 33u, Capacitor_SMD:CP_Elec_10x10
- C5: value 33u -> 100u
- moved U3 212.6 mm to (257.5, 104.4)
- moved U2 177.0 mm to (186.0, 140.0)
- moved U5 173.9 mm to (240.7, 39.3)
- moved C2 124.5 mm to (89.5, 175.0)
- moved R5 120.7 mm to (206.5, 101.0)
- moved C3 119.9 mm to (92.0, 186.5)
- moved F1 115.3 mm to (143.1, 136.2)
- moved L1 112.7 mm to (71.0, 179.0), turned to -90 degrees
- moved U4 112.1 mm to (208.7, 47.5)
- moved R3 109.6 mm to (208.0, 106.5)
- moved BT1 104.5 mm to (159.0, 74.5), turned to 180 degrees
- moved U1 102.2 mm to (94.5, 163.5)
- moved C1 97.1 mm to (71.0, 157.5), turned to 90 degrees
- moved M2 96.0 mm to (167.5, 30.0)
- moved D5 91.7 mm to (143.3, 144.6)
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Other:
- rule pad_to_mask_clearance: 0 -> 0.0508

Commit message: Layout and routing
Parts:
- removed the C5 at (156.0, 85.0)
- moved U3 146.1 mm to (113.9, 77.4)
- moved F1 128.7 mm to (31.5, 72.0), turned to 90 degrees
- moved D4 128.7 mm to (37.0, 72.0), turned to 90 degrees
- moved R4 125.2 mm to (91.8, 60.0), turned to 180 degrees
- moved U5 123.7 mm to (124.1, 80.7), turned to -90 degrees
- moved BT1 123.0 mm to (36.5, 63.0)
- moved R5 118.7 mm to (93.2, 65.5), turned to 180 degrees
- moved U2 109.9 mm to (82.1, 104.4)
- moved M1 104.5 mm to (72.5, 58.2)
- moved M2 103.7 mm to (67.8, 58.2)
- moved R6 102.6 mm to (46.5, 54.0), turned to -90 degrees
- moved C5 102.0 mm to (58.2, 51.0)
- moved J1 101.9 mm to (37.1, 53.1), turned to 90 degrees
- moved R7 101.6 mm to (46.5, 57.0), turned to 90 degrees
- moved J2 90.3 mm to (59.5, 42.5)
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- renumbered C8 to C5, C9 to C6, D2 to D1, D3 to D2, D4 to D3, D5 to D4, D1 to D5, R4 to R3, R3 to R4
Connections:
- J1 pad 1: Net-(J1-Pad1) -> /RX_P
- J1 pad 2: Net-(J1-Pad2) -> /RX_N
- J1 pad 3: Net-(J1-Pad3) -> GND
- J1 pad 4: +24V -> GND
- J1 pad 6: Net-(J1-Pad6) -> +24V
- J1 pad 7: GND -> /TX_P
- J1 pad 8: GND -> /TX_N
- R6 pad 1: Net-(J1-Pad6) -> /TX_P
- R6 pad 2: Net-(J1-Pad3) -> /TX_N
- R7 pad 1: Net-(J1-Pad2) -> /RX_P
- R7 pad 2: Net-(J1-Pad1) -> /RX_N
- U2 pad 6: unconnected-(U2-Pad6) -> /ARGB_DATA
- U6 pad 5: Net-(J1-Pad6) -> /TX_P
- U6 pad 6: Net-(J1-Pad3) -> /TX_N
- U6 pad 7: Net-(J1-Pad1) -> /RX_N
- U6 pad 8: Net-(J1-Pad2) -> /RX_P
- U7 pad 2: unconnected-(U7-Pad2) -> /ARGB_DATA
Routing:
- net GND: track 0.00 -> 91.6 mm, vias 0 -> 1
- net +24V: track 0.00 -> 21.4 mm
- net /TX_N: track 0.00 -> 18.1 mm
- net /TX_P: track 0.00 -> 18.0 mm
- net +5V: track 0.00 -> 15.4 mm
- net /RX_P: track 0.00 -> 14.0 mm
- net /RX_N: track 0.00 -> 13.9 mm
- net +3V3: track 0.00 -> 13.4 mm
- net Net-(D3-Pad1): track 0.00 -> 2.27 mm
- net Net-(D2-Pad1): track 0.00 -> 2.27 mm
- net Net-(D1-Pad1): track 0.00 -> 2.27 mm
- added copper zone on F.Cu, net +24V
- added copper zone on F.Cu, net +5V
- added copper zone on F.Cu, net GND
- added copper zone on F.Cu, net Net-(C1-Pad1)
- added copper zone on F.Cu, net Net-(D5-Pad1)

Commit message: "done" but ugly
Parts:
- moved R4 4.42 mm to (95.4, 62.5), turned to 0 degrees
- moved R5 2.19 mm to (95.4, 65.1), turned to 0 degrees
- moved J2 1.00 mm to (59.5, 41.5)
Connections:
- U2 pad 4: /SRV1_PWM -> /SRV2_PWM
- U2 pad 5: /SRV2_PWM -> /SRV1_PWM
Routing:
- net +5V: track 15.4 -> 182.5 mm, vias 0 -> 2
- net +3V3: track 13.4 -> 153.0 mm, vias 0 -> 2
- net /SDA: track 0.00 -> 55.2 mm, vias 0 -> 2
- net /SCL: track 0.00 -> 55.2 mm, vias 0 -> 2
- net /COMMS_RST: track 0.00 -> 40.4 mm
- net /COMMS_G0: track 0.00 -> 37.5 mm
- net /COMMS_CS: track 0.00 -> 35.4 mm
- net /COMP_TX: track 0.00 -> 33.2 mm, vias 0 -> 2
- net /GPS_RX: track 0.00 -> 32.3 mm, vias 0 -> 2
- net /COMP_RX: track 0.00 -> 32.0 mm, vias 0 -> 2
- net /MOSI: track 0.00 -> 31.9 mm
- net /GPS_TX: track 0.00 -> 31.2 mm, vias 0 -> 2
- net /MISO: track 0.00 -> 29.7 mm
- net /ARGB_DATA: track 0.00 -> 25.0 mm, vias 0 -> 2
- net /SRV2_PWM: track 0.00 -> 19.7 mm
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- added copper zone on B.Cu, net GND
Other:
- board outline added: 123 x 74 mm

Commit message: Working on PCB
Parts:
- added H1: MountingHole_Pad, MountingHole:MountingHole_3.2mm_M3_Pad, F.Cu at (35.0, 87.5)
- added H2: MountingHole_Pad, MountingHole:MountingHole_3.2mm_M3_Pad, F.Cu at (145.0, 37.5)
- added H3: MountingHole_Pad, MountingHole:MountingHole_3.2mm_M3_Pad, F.Cu at (35.0, 37.5)
- added H4: MountingHole_Pad, MountingHole:MountingHole_3.2mm_M3_Pad, F.Cu at (145.0, 87.5)
- added J3: QWIIC_Generic_Conn, Connector_JST:JST_SH_BM04B-SRSS-TB_1x04-1MP_P1.00mm_Vertical, F.Cu at (150.5, 46.5)
- moved BT1 27.8 mm to (47.5, 37.5)
- moved U4 11.9 mm to (149.5, 66.5)
- moved C3 11.6 mm to (74.8, 96.5)
- moved C2 11.4 mm to (71.8, 84.5)
- moved L1 10.4 mm to (53.5, 91.5)
- moved D1 8.35 mm to (55.8, 44.0)
- moved D2 8.35 mm to (55.8, 39.8)
- moved D3 8.35 mm to (55.8, 35.5)
- moved R1 8.04 mm to (57.6, 44.0)
- moved R2 8.04 mm to (57.6, 39.8)
- moved R3 8.04 mm to (57.6, 35.5)
- moved C1 6.71 mm to (48.0, 67.0)
- moved C4 6.71 mm to (56.5, 53.0)
- moved C5 6.71 mm to (61.2, 45.0)
- moved C6 6.71 mm to (78.0, 36.0)
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Routing:
- net +3V3: track 153.0 -> 176.6 mm
- net +24V: track 21.4 -> 44.8 mm
- net GND: track 91.6 -> 70.6 mm, vias 1 -> 145
- net /SDA: track 55.2 -> 73.1 mm
- net /SCL: track 55.2 -> 68.3 mm
- net /RX_P: track 14.0 -> 19.5 mm
- net /RX_N: track 13.9 -> 19.3 mm
- net +5V: track 182.5 -> 180.2 mm
- net /TX_N: track 18.1 -> 19.7 mm
- net /TX_P: track 18.0 -> 19.6 mm
Other:
- outline, holes or cut-outs redrawn
- board text added: "3.3V"
- board text added: "5V"
- board text added: "Vin"

Commit message: Changes
Parts:
- removed H3, H4: MountingHole_Pad, MountingHole:MountingHole_3.2mm_M3_Pad
- added G***: LOGO, ASTRA_Footprints:SHCLogo, B.Cu at (114.0, 118.0)
- added G***: LOGO, ASTRA_Footprints:ATRALogo, B.Cu at (195.5, 80.5)
- H1, H2: footprint MountingHole:MountingHole_3.2mm_M3_Pad -> MountingHole:MountingHole_4.3mm_M4_Pad
- moved J3 100.7 mm to (204.5, 131.5), turned to 180 degrees
- moved H2 87.8 mm to (209.5, 97.0)
- moved U4 82.4 mm to (213.5, 118.5)
- moved BT1 73.8 mm to (108.0, 79.8)
- moved C4 71.0 mm to (120.8, 83.2)
- moved R6 71.0 mm to (113.8, 78.2)
- moved R7 71.0 mm to (113.8, 81.2)
- moved U6 71.0 mm to (118.8, 79.8)
- moved D4 70.3 mm to (107.5, 85.5), turned to 0 degrees
- moved C1 68.7 mm to (111.0, 94.5)
- moved C2 68.7 mm to (134.8, 112.0)
- moved C3 68.7 mm to (137.8, 124.0)
- moved C5 68.7 mm to (124.2, 72.5)
- moved C6 68.7 mm to (141.0, 63.5)
- moved D1 68.7 mm to (118.8, 71.5)
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Connections:
- BT1 pad 2: +24V -> /Power_in
- C1 pad 1: Net-(C1-Pad1) -> +24V
- D4 pad 1: Net-(C1-Pad1) -> +24V
- F1 pad 1: Net-(C1-Pad1) -> +24V
- F1 pad 2: +24V -> /Power_in
- J1 pad 3: GND -> /Power_in
- J1 pad 4: GND -> /Power_in
- J1 pad 5: +24V -> GND
- J1 pad 6: +24V -> GND
- U1 pad 1: Net-(C1-Pad1) -> +24V
Routing:
- net +24V: track 44.8 -> 70.4 mm, vias 0 -> 2
- net /SCL: track 68.3 -> 93.8 mm, vias 2 -> 3
- net /Power_in: track 0.00 -> 19.3 mm
- net /SDA: track 73.1 -> 91.2 mm, vias 2 -> 3
- net GND: track 70.6 -> 59.5 mm, vias 145 -> 134
- net /RX_N: track 19.3 -> 26.0 mm, vias 0 -> 1
- net /RX_P: track 19.5 -> 26.3 mm, vias 0 -> 1
- net /TX_P: track 19.6 -> 26.0 mm, vias 0 -> 1
- net /TX_N: track 19.7 -> 25.7 mm, vias 0 -> 1
- net +3V3: track 176.6 -> 171.6 mm
- net +5V: track 180.2 -> 177.1 mm
- net /ARGB_DATA: track 25.0 -> 26.2 mm
- added copper zone on F.Cu, net /Power_in
- removed copper zone on F.Cu, net Net-(C1-Pad1)
Other:
- board text added: "UAH SHC ASTRA Base Station PCB V1 April 2022"
