File: Ground_Station_Electronics/Ground_Station_Electronics.kicad_pcb (KiCad board)
At the start: 2 copper layers, 123 x 74 mm, 37 parts, among them J1 RJ45_Shielded_Labelled, J2 ARGB_Header, J3 QWIIC_Generic_Conn, M1 Motor_Servo, M2 Motor_Servo, U1 LM2576HVS-5, U2 Teensy_4.1, U3 Adafruit_GPS_V3, U4 BNO055_Adafruit_Breakout, U5 RFM95W_Adafruit_Breakout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

Commit message: Updated, ready to order
Connections:
- J1 pad SH: GND -> unconnected-(J1-PadSH)
Changed lines of the file:
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@@
   (net 75 "unconnected-(H1-Pad1)")
   (net 76 "unconnected-(H2-Pad1)")
+  (net 77 "unconnected-(J1-PadSH)")
   (footprint "ASTRA_Footprints:Teensy4.1" (layer "F.Cu")
     (at 148.0625 125.885)
@@
       (net 12 "/TX_N") (pinfunction "BRN") (pintype "passive"))
     (pad "SH" thru_hole circle (at -4.57 0.89) (size 2.3 2.3) (drill 1.57) (layers *.Cu *.Mask)
-      (net 1 "GND") (pintype "passive"))
+      (net 77 "unconnected-(J1-PadSH)") (pintype "passive"))
     (pad "SH" thru_hole circle (at 11.69 0.89) (size 2.3 2.3) (drill 1.57) (layers *.Cu *.Mask)
-      (net 1 "GND") (pintype "passive"))
+      (net 77 "unconnected-(J1-PadSH)") (pintype "passive"))
     (model "${KICAD6_3DMODEL_DIR}/Connector_RJ.3dshapes/RJ45_Amphenol_RJHSE5380.wrl"
       (offset (xyz 0 0 0))
