File: Ground_Station_Dongle/Ground_Station_Dongle.kicad_pcb (KiCad board)
At the start: 2 copper layers, 44 x 20 mm, 15 parts, among them J51 USB_UART_Header, J52 RJ45_Shielded_Labelled, J53 Barrel_Jack_MountingPin, U51 MAX3488E

Commit message: Updated, ready to order
Parts:
- removed JP51, JP54: SolderJumper_2_Bridged, Jumper:SolderJumper-2_P1.3mm_Bridged_RoundedPad1.0x1.5mm
- removed JP52, JP53: SolderJumper_2_Open, Jumper:SolderJumper-2_P1.3mm_Open_RoundedPad1.0x1.5mm
- added G***: LOGO, LOGO, B.Cu at (61.0, 27.0)
- moved R53 6.40 mm to (64.9, 23.5), turned to 180 degrees
- moved R54 6.20 mm to (61.9, 23.5), turned to 0 degrees
- moved C51 5.68 mm to (59.9, 30.0), turned to -90 degrees
- moved U51 1.19 mm to (63.4, 28.5), turned to 90 degrees
- moved J51 0.65 mm to (84.0, 20.6)
Connections:
- J51 pad 2: unconnected-(J51-Pad2) -> GND
- J51 pad 4: Net-(J51-Pad4) -> /COMP_RX
- J51 pad 5: Net-(J51-Pad5) -> /COMP_TX
- J52 pad 1: /RX_P -> /TX_P
- J52 pad 2: /RX_N -> /TX_N
- J52 pad 7: /TX_P -> /RX_P
- J52 pad 8: /TX_N -> /RX_N
Routing:
- net Net-(J51-Pad4): track 21.4 -> 0.00 mm, vias 1 -> 0
- net Net-(J51-Pad5): track 16.4 -> 0.00 mm, vias 1 -> 0
- net /Power_in: track 32.5 -> 48.8 mm
- net /COMP_RX: track 14.9 -> 28.6 mm, vias 1 -> 0
- net /COMP_TX: track 15.6 -> 22.6 mm, vias 1 -> 0
- net /RX_P: track 11.9 -> 17.4 mm
- net /RX_N: track 11.6 -> 17.1 mm
- net /TX_P: track 14.1 -> 19.5 mm
- net /TX_N: track 14.1 -> 19.3 mm
- net +3V3: track 35.0 -> 38.2 mm
Other:
- board text added: "2.1x5.5"
- board text added: "24V IN"
- board text added: "RS485 over RJ45 NOT ETHERNET!!"
- board text added: "UAH SHC ASTRA Ground Station Dongle V1 Apr 2022"
