File: Ground_Station_Dongle/Ground_Station_Dongle.kicad_sch (KiCad schematic)
At the start: 15 parts

Commit message: Updated, ready to order
Parts:
- removed JP51, JP54: (no value), symbol Jumper:SolderJumper_2_Bridged
- removed JP52, JP53: (no value), symbol Jumper:SolderJumper_2_Open
- C51: value (none) -> 100n; footprint (none) -> Capacitor_SMD:C_0603_1608Metric
- D51, D52: value (none) -> G; footprint (none) -> LED_SMD:LED_0603_1608Metric_Pad1.05x0.95mm_HandSolder
- J52: value (none) -> RJ45_Shielded_Labelled; footprint (none) -> Connector_RJ:RJ45_Amphenol_RJHSE5380
- J53: value (none) -> Barrel_Jack_MountingPin; footprint (none) -> Connector_BarrelJack:BarrelJack_CUI_PJ-063AH_Horizontal; Digikey Part Num (none) -> CP-063AH-ND
- R51: value (none) -> 10; footprint (none) -> Resistor_SMD:R_0603_1608Metric
- R52: value (none) -> 3.3k; footprint (none) -> Resistor_SMD:R_0603_1608Metric
- R53, R54: value (none) -> 120; footprint (none) -> Resistor_SMD:R_0603_1608Metric
Connections:
- net COMP_RX: now also J51.4 (RXI)
- net COMP_TX: now also J51.5 (TXO)
- net GND: now also J51.2 (CTS)
- no-connect marks 2 -> 1
Other:
- moved on the sheet: J52
